File: PCB/Macro Pad.kicad_pcb (KiCad board)
At the start: 2 copper layers, 84.4 x 41.2 mm, 11 parts, among them SW1 SW_Push, SW2 SW_Push, SW3 SW_Push, SW4 SW_Push, SW5 SW_Push, SW6 SW_Push, SW7 RotaryEncoder_Switch, U1 XIAO-RP2040-DIP

Commit message: Update files
Parts:
- removed D1, D2, D3: SK6812MINI, LED_SMD:LED_SK6812MINI_PLCC4_3.5x3.5mm_P1.75mm
- added D4: SK6812MINI-E, Hackclub Footprints:MX_SK6812MINI-E_REV, B.Cu at (203.6, 50.1)
- added D5: SK6812MINI-E, Hackclub Footprints:MX_SK6812MINI-E_REV, B.Cu at (203.6, 43.4)
- added D6: SK6812MINI-E, Hackclub Footprints:MX_SK6812MINI-E_REV, B.Cu at (203.6, 37.4)
Routing:
- net Net-(D4-DIN): track 6.35 -> 33.7 mm, vias 0 -> 2
- net Net-(D4-DOUT): track 0.00 -> 19.9 mm, vias 0 -> 2
- net Net-(D5-DOUT): track 0.00 -> 19.5 mm, vias 0 -> 2
- net Net-(D1-DOUT): track 13.0 -> 0.00 mm, vias 2 -> 0
- net Net-(D2-DOUT): track 12.0 -> 0.00 mm, vias 2 -> 0
- net +5V: track 23.7 -> 32.0 mm
- net GND: track 179.5 -> 183.2 mm
- net Net-(U1-GPIO7/SCL): track 87.5 -> 90.8 mm
