File: PCB/Macro Pad.kicad_sch (KiCad schematic)
At the start: 11 parts, among them SW1 SW_Push, SW2 SW_Push, SW3 SW_Push, SW4 SW_Push, SW5 SW_Push, SW6 SW_Push, SW7 RotaryEncoder_Switch, U1 XIAO-RP2040-DIP

Commit message: Update files
Parts:
- removed D1, D2, D3: SK6812MINI, LED_SMD:LED_SK6812MINI_PLCC4_3.5x3.5mm_P1.75mm, symbol LED:SK6812MINI
- added D4, D5, D6: SK6812MINI-E, Hackclub Footprints:MX_SK6812MINI-E_REV, symbol Hackclub Symbols:SK6812MINI-E
Connections:
- net +5V: now also D4.1 (VDD), D5.1 (VDD), D6.1 (VDD)
- net GND: now also D4.3 (VSS), D5.3 (VSS), D6.3 (VSS)
- net at U1.1 (GPIO26/ADC0/A0): now also D4.4 (DIN)
- new net: D5.2 (DOUT), D6.4 (DIN)
- new net: D4.2 (DOUT), D5.4 (DIN)
